File: cassy/cassy.kicad_sch (KiCad schematic)
At the start: 3 parts, among them J1 DB15_Male, J2 Conn_01x03_Male, U1 MAX4659

Commit message: change layer
Parts:
- added C1, C2: C, Capacitor_SMD:C_0805_2012Metric, symbol Device:C
Connections:
- net +12V: now also C2.2
- net -12V: now also C1.1
- net GND: now also C1.2, C2.1
Changed lines of the file:
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@@
   (junction (at 120.65 81.28) (diameter 0) (color 0 0 0 0)
   )
+  (junction (at 180.34 86.36) (diameter 0) (color 0 0 0 0)
+  )
   (junction (at 120.65 101.6) (diameter 0) (color 0 0 0 0)
   )
+  (junction (at 175.26 86.36) (diameter 0) (color 0 0 0 0)
+  )
   (junction (at 120.65 91.44) (diameter 0) (color 0 0 0 0)
   )
@@
     (stroke (width 0) (type default))
   )
+  (wire (pts (xy 189.23 86.36) (xy 190.5 86.36))
+    (stroke (width 0) (type default))
+  )
   (wire (pts (xy 120.65 96.52) (xy 120.65 91.44))
     (stroke (width 0) (type default))
@@
     (stroke (width 0) (type default))
   )
+  (wire (pts (xy 165.1 86.36) (xy 166.37 86.36))
+    (stroke (width 0) (type default))
+  )
   (wire (pts (xy 118.11 101.6) (xy 120.65 101.6))
     (stroke (width 0) (type default))
   )
-  (wire (pts (xy 175.26 85.09) (xy 175.26 87.63))
-    (stroke (width 0) (type default))
-  )
-  (wire (pts (xy 180.34 85.09) (xy 180.34 87.63))
+  (wire (pts (xy 175.26 85.09) (xy 175.26 86.36))
+    (stroke (width 0) (type default))
+  )
+  (wire (pts (xy 180.34 85.09) (xy 180.34 86.36))
     (stroke (width 0) (type default))
   )
@@
     (stroke (width 0) (type default))
   )
+  (wire (pts (xy 175.26 86.36) (xy 175.26 87.63))
+    (stroke (width 0) (type default))
+  )
+  (wire (pts (xy 180.34 86.36) (xy 181.61 86.36))
+    (stroke (width 0) (type default))
+  )
   (wire (pts (xy 118.11 83.82) (xy 158.75 83.82))
     (stroke (width 0) (type default))
@@
     (stroke (width 0) (type default))
   )
+  (wire (pts (xy 180.34 86.36) (xy 180.34 87.63))
+    (stroke (width 0) (type default))
+  )
   (wire (pts (xy 120.65 111.76) (xy 120.65 106.68))
     (stroke (width 0) (type default))
@@
   )
   (wire (pts (xy 118.11 99.06) (xy 120.65 99.06))
+    (stroke (width 0) (type default))
+  )
+  (wire (pts (xy 173.99 86.36) (xy 175.26 86.36))
     (stroke (width 0) (type default))
   )
@@
     )
   )
+  (symbol (lib_id "Device:C") (at 185.42 86.36 90) (unit 1)
+    (in_bom yes) (on_board yes) (dnp no) (fields_autoplaced)
+    (property "Reference" "C1" (at 185.42 80.01 90)
+      (effects (font (size 1.27 1.27)))
+    )
+    (property "Value" "C" (at 185.42 82.55 90)
+      (effects (font (size 1.27 1.27)))
+    )
+    (property "Footprint" "Capacitor_SMD:C_0805_2012Metric" (at 189.23 85.3948 0)
+      (effects (font (size 1.27 1.27)) hide)
+    )
+    (property "Datasheet" "~" (at 185.42 86.36 0)
+      (effects (font (size 1.27 1.27)) hide)
+    )
+    (pin "1")
+    (pin "2")
+    (instances
+      (project "cassy"
+        (path "/9861448e-4d91-44d5-a7ed-c342cf9a199e"
+          (reference "C1") (unit 1)
+        )
+      )
+    )
+  )
   (symbol (lib_id "power:+12V") (at 121.92 86.36 270) (unit 1)
     (in_bom yes) (on_board yes) (dnp no) (fields_autoplaced)
@@
     )
   )
+  (symbol (lib_id "power:GND") (at 190.5 86.36 90) (unit 1)
+    (in_bom yes) (on_board yes) (dnp no) (fields_autoplaced)
+    (property "Reference" "#PWR08" (at 196.85 86.36 0)
+      (effects (font (size 1.27 1.27)) hide)
+    )
+    (property "Value" "GND" (at 194.31 86.995 90)
+      (effects (font (size 1.27 1.27)) (justify right))
+    )
+    (property "Footprint" "" (at 190.5 86.36 0)
+      (effects (font (size 1.27 1.27)) hide)
+    )
+    (property "Datasheet" "" (at 190.5 86.36 0)
+      (effects (font (size 1.27 1.27)) hide)
+    )
+    (pin "1")
+    (instances
+      (project "cassy"
+        (path "/9861448e-4d91-44d5-a7ed-c342cf9a199e"
+          (reference "#PWR08") (unit 1)
+        )
+      )
+    )
+  )
   (symbol (lib_id "power:GND") (at 177.8 110.49 0) (unit 1)
     (in_bom yes) (on_board yes) (dnp no) (fields_autoplaced)
@@
         (path "/9861448e-4d91-44d5-a7ed-c342cf9a199e"
           (reference "#PWR02") (unit 1)
+        )
+      )
+    )
+  )
+  (symbol (lib_id "power:GND") (at 165.1 86.36 270) (unit 1)
+    (in_bom yes) (on_board yes) (dnp no) (fields_autoplaced)
+    (property "Reference" "#PWR09" (at 158.75 86.36 0)
+      (effects (font (size 1.27 1.27)) hide)
+    )
+    (property "Value" "GND" (at 161.29 86.995 90)
+      (effects (font (size 1.27 1.27)) (justify right))
+    )
+    (property "Footprint" "" (at 165.1 86.36 0)
+      (effects (font (size 1.27 1.27)) hide)
+    )
+    (property "Datasheet" "" (at 165.1 86.36 0)
+      (effects (font (size 1.27 1.27)) hide)
+    )
+    (pin "1")
+    (instances
+      (project "cassy"
+        (path "/9861448e-4d91-44d5-a7ed-c342cf9a199e"
+          (reference "#PWR09") (unit 1)
         )
       )
@@
         )
       )
+    )
+  )
+  (symbol (lib_id "Device:C") (at 170.18 86.36 90) (unit 1)
+    (in_bom yes) (on_board yes) (dnp no) (fields_autoplaced)
+    (property "Reference" "C2" (at 170.18 80.01 90)
+      (effects (font (size 1.27 1.27)))
+    )
+    (property "Value" "C" (at 170.18 82.55 90)
+      (effects (font (size 1.27 1.27)))
+    )
+    (property "Footprint" "Capacitor_SMD:C_0805_2012Metric" (at 173.99 85.3948 0)
+      (effects (font (size 1.27 1.27)) hide)
+    )
+    (property "Datasheet" "~" (at 170.18 86.36 0)
+      (effects (font (size 1.27 1.27)) hide)
+    )
+    (pin "1")
+    (pin "2")
+    (instances
+      (project "cassy"
+        (path "/9861448e-4d91-44d5-a7ed-c342cf9a199e"
+          (reference "C2") (unit 1)
+        )
+      )

Commit message: insert PDF
Other:
- company: (none) -> elektrotechnik2go.de
- title: (none) -> Cassy
Changed lines of the file:
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@@
 (kicad_sch (version 20230121) (generator eeschema)
   (paper "A4")
+  (title_block
+    (title "Cassy")
+    (date "2023-06-05")
+    (company "elektrotechnik2go.de")
+    (comment 1 "Johann Schmid")
+  )
   (junction (at 120.65 81.28) (diameter 0) (color 0 0 0 0)
   )
