File: cassy/cassy.kicad_sch (KiCad schematic)
At the start: 18 parts, among them J1 DB15_Male, J2 Conn_01x03_Male, U1 MAX4659, U2 OPA2202

Commit message: update
Parts:
- C6: value C_Polarized -> 100u
Changed lines of the file:
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@@
       (effects (font (size 1.27 1.27)) (justify right))
     )
-    (property "Value" "C_Polarized" (at 251.46 131.699 0)
+    (property "Value" "100u" (at 251.46 131.699 0)
       (effects (font (size 1.27 1.27)) (justify right))
     )

Commit message: update PCB
update
Parts:
- U1: footprint Package_SO:MSOP-8_3x3mm_P0.65mm -> Package_SO:SOIC-8_3.9x4.9mm_P1.27mm
- U2: footprint Package_SO:SOIC-8_3.9x4.9mm_P1.27mm -> Package_SO:MSOP-8_3x3mm_P0.65mm
Changed lines of the file:
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@@
       (effects (font (size 1.27 1.27)))
     )
-    (property "Footprint" "Package_SO:SOIC-8_3.9x4.9mm_P1.27mm" (at 102.87 96.52 0)
+    (property "Footprint" "Package_SO:MSOP-8_3x3mm_P0.65mm" (at 102.87 96.52 0)
       (effects (font (size 1.27 1.27)) hide)
     )
@@
       (effects (font (size 1.27 1.27)))
     )
-    (property "Footprint" "Package_SO:SOIC-8_3.9x4.9mm_P1.27mm" (at 104.14 137.16 0)
+    (property "Footprint" "Package_SO:MSOP-8_3x3mm_P0.65mm" (at 104.14 137.16 0)
       (effects (font (size 1.27 1.27)) hide)
     )
@@
       (effects (font (size 1.27 1.27)))
     )
-    (property "Footprint" "Package_SO:SOIC-8_3.9x4.9mm_P1.27mm" (at 222.25 129.54 0)
+    (property "Footprint" "Package_SO:MSOP-8_3x3mm_P0.65mm" (at 222.25 129.54 0)
       (effects (font (size 1.27 1.27)) hide)
     )
@@
       (effects (font (size 1.27 1.27)))
     )
-    (property "Footprint" "Package_SO:MSOP-8_3x3mm_P0.65mm" (at 190.5 92.71 0)
-      (effects (font (size 1.27 1.27)) hide)
-    )
+    (property "Footprint" "Package_SO:SOIC-8_3.9x4.9mm_P1.27mm" (at 190.5 92.71 0)
+      (effects (font (size 1.27 1.27)) hide)
+    )
