File: cassy/cassy.kicad_pcb (KiCad board)
At the start: 2 copper layers, 36.9 x 40.2 mm, 3 parts, among them J1 DB15_Male, J2 Conn_01x03_Male, U1 MAX4659

Commit message: change layer
Parts:
- added ?: , , F.Cu at (87.7, 104.6)
- added ?: , , F.Cu at (91.6, 104.7)
- added C1: C, Capacitor_SMD:C_0805_2012Metric, F.Cu at (83.9, 104.6)
- added C2: C, Capacitor_SMD:C_0805_2012Metric, F.Cu at (91.9, 97.2)
- J1, J2: moved to B.Cu
- moved J1 19.6 mm to (79.7, 109.8), turned to 90 degrees
- turned J2 to 0 degrees
Routing:
- net -12V: track 19.8 -> 14.4 mm
- net Net-(J2-Pin_1): track 16.2 -> 13.0 mm
- net Net-(J1-P9): track 23.1 -> 20.2 mm
- net +12V: track 21.8 -> 20.3 mm
- net IN: track 11.5 -> 12.3 mm
- net GND: track 0.64 -> 0.00 mm

Commit message: insert pdf layout
Other:
- board text added: "github.com/ Johann-Schmid/Cassy www.elektrotechnik2go.de"
Changed lines of the file:
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@@
   (gr_rect (start 66.69 79.67) (end 103.61 119.86)
     (stroke (width 0.1) (type default)) (fill none) (layer "Edge.Cuts"))
+  (gr_text "github.com/\nJohann-Schmid/Cassy\n\nwww.elektrotechnik2go.de" (at 83 91.98) (layer "F.Cu")
+    (effects (font (size 1 1) (thickness 0.2) bold) (justify left bottom))
+  )
   (segment (start 91.9325 100.025) (end 89.445 100.025) (width 0.4) (layer "F.Cu") (net 2))
   (segment (start 88.125 106.985) (end 79.68 106.985) (width 0.4) (layer "F.Cu") (net 2))
@@
   (segment (start 96.315 101.325) (end 97.75 102.76) (width 0.4) (layer "F.Cu") (net 11))
   (zone (net 1) (net_name "GND") (layer "F.Cu") (hatch edge 0.5)
-    (connect_pads (clearance 0.2))
-    (min_thickness 0.2) (filled_areas_thickness no)
+    (connect_pads (clearance 0.3))
+    (min_thickness 0.3) (filled_areas_thickness no)
     (fill yes (thermal_gap 0.5) (thermal_bridge_width 0.5))
     (polygon

Commit message: insert op2202
Parts:
- removed ? (x2): , 
- added C3: 100n, Capacitor_SMD:C_0805_2012Metric, F.Cu at (119.7, 95.5)
- added C4: 100n, Capacitor_SMD:C_0805_2012Metric, F.Cu at (99.0, 103.9)
- added C5: 100u, Capacitor_THT:CP_Radial_D6.3mm_P2.50mm, F.Cu at (113.7, 95.6)
- added C6: C_Polarized, Capacitor_THT:CP_Radial_D6.3mm_P2.50mm, F.Cu at (93.5, 112.8)
- added R1: 390k, Resistor_SMD:R_0805_2012Metric_Pad1.20x1.40mm_HandSolder, F.Cu at (114.7, 111.5)
- added R2: 1k, Resistor_SMD:R_0805_2012Metric_Pad1.20x1.40mm_HandSolder, F.Cu at (97.8, 99.3)
- added R3: 100, Resistor_SMD:R_0805_2012Metric_Pad1.20x1.40mm_HandSolder, F.Cu at (97.8, 91.7)
- added R4: 390k, Resistor_SMD:R_0805_2012Metric_Pad1.20x1.40mm_HandSolder, F.Cu at (115.1, 84.0)
- added R5: 1k, Resistor_SMD:R_0805_2012Metric_Pad1.20x1.40mm_HandSolder, F.Cu at (111.1, 101.4)
- added R6: 100, Resistor_SMD:R_0805_2012Metric_Pad1.20x1.40mm_HandSolder, F.Cu at (115.2, 102.7)
- added RV1: 100k, Potentiometer_THT:Potentiometer_ACP_CA9-H2,5_Horizontal, F.Cu at (108.0, 111.5)
- added RV2: 100k, Potentiometer_THT:Potentiometer_ACP_CA9-H2,5_Horizontal, F.Cu at (107.5, 84.1)
- added U2: OPA2202, Package_SO:SOIC-8_3.9x4.9mm_P1.27mm, F.Cu at (104.2, 100.8)
- C1, C2: value C -> 100n
- moved J2 26.5 mm to (123.3, 98.4)
- moved C2 17.1 mm to (108.2, 91.7)
- moved C1 2.41 mm to (85.3, 106.6), turned to -90 degrees
Connections:
- U1 pad 2: Net-(J2-Pin_2) -> Net-(U1-NC)
- U1 pad 8: Net-(J2-Pin_1) -> Net-(U1-NO)
Routing:
- net +12V: track 20.3 -> 88.3 mm, vias 0 -> 2
- net -12V: track 14.4 -> 76.6 mm
- net Net-(J1-P9): track 20.2 -> 66.3 mm
- net Net-(U1-NC): track 0.00 -> 37.0 mm, vias 0 -> 2
- net Net-(U1-NO): track 0.00 -> 29.7 mm
- net Net-(U2B-+): track 0.00 -> 17.8 mm
- net GND: track 0.00 -> 17.1 mm, vias 0 -> 2
- net Net-(J2-Pin_2): track 6.41 -> 23.1 mm
- net Net-(U2A-+): track 0.00 -> 15.3 mm
- net Net-(R4-Pad2): track 0.00 -> 6.77 mm
- net Net-(R1-Pad2): track 0.00 -> 5.81 mm
- net Net-(U2A--): track 0.00 -> 5.34 mm
- net Net-(J2-Pin_1): track 13.0 -> 18.0 mm
- net Net-(U2B--): track 0.00 -> 4.80 mm
Other:
- board size 36.9 x 40.2 mm -> 61.7 x 40.2 mm

Commit message: update PCB
update
Parts:
- C6: value C_Polarized -> 100u
- U1: footprint Package_SO:MSOP-8_3x3mm_P0.65mm -> Package_SO:SOIC-8_3.9x4.9mm_P1.27mm
- U2: footprint Package_SO:SOIC-8_3.9x4.9mm_P1.27mm -> Package_SO:MSOP-8_3x3mm_P0.65mm
- moved U2 0.82 mm to (104.5, 100.0)
- moved U1 0.17 mm to (89.7, 101.0)
Routing:
- net -12V: track 76.6 -> 78.8 mm
- net Net-(U2B-+): track 17.8 -> 15.9 mm
- net IN: track 12.3 -> 13.2 mm
- net Net-(J1-P9): track 66.3 -> 67.1 mm
- net Net-(U1-NO): track 29.7 -> 29.0 mm
- net +12V: track 88.3 -> 87.7 mm
